File: pcb/oven_pcb/oven_pcb.kicad_pcb (KiCad board)
At the start: 2 copper layers, 16 parts

Commit message: pcb_v2
Parts:
- removed REF** (x14): Pin_D0.9mm_L10.0mm_W2.4mm_FlatFork, Connector_Pin:Pin_D0.9mm_L10.0mm_W2.4mm_FlatFork
- removed REF**: yautay-5V-stepdown, Converter_DCDC:yautay-5V-stepdown
- removed REF**: nodeMCUv3, Module:nodeMCUv3
- added 100k1: R, Resistor_THT:R_Axial_DIN0207_L6.3mm_D2.5mm_P10.16mm_Horizontal, F.Cu at (89.9, 70.1)
- added NTC1: Conn_01x02_Male, Connector_PinHeader_2.54mm:PinHeader_1x02_P2.54mm_Vertical, F.Cu at (84.8, 79.0)
- added PSU1: Conn_01x02_Male, Connector_PinHeader_2.54mm:PinHeader_1x02_P2.54mm_Vertical, F.Cu at (88.9, 118.1)
- added U1: D24V10F5, Converter_DCDC:yautay-5V-stepdown, F.Cu at (94.0, 110.7)
- added U2: NodeMCU_3.0_(ESP-12E), Module:nodeMCUv3, F.Cu at (114.6, 80.3)
- added U3: SSR, Connector_PinHeader_2.54mm:PinHeader_1x02_P2.54mm_Vertical, F.Cu at (134.6, 87.9)
- added yautay1: BME2803V, Connector_PinHeader_2.54mm:PinHeader_1x06_P2.54mm_Vertical, F.Cu at (134.9, 67.6)
Routing:
- net (no net): track 325.4 -> 269.2 mm
- net Net-(U2-Pad16): track 0.00 -> 52.9 mm
- net Net-(NTC1-Pad2): track 0.00 -> 27.5 mm
- net Net-(100k1-Pad1): track 0.00 -> 20.4 mm
- net +24V: track 0.00 -> 12.4 mm
- net Net-(U1-Pad5): track 0.00 -> 7.87 mm
- net Net-(U2-Pad29): track 0.00 -> 7.63 mm
- net Net-(U2-Pad28): track 0.00 -> 7.63 mm
- net Net-(U2-Pad23): track 0.00 -> 7.37 mm
- added copper zone on B.Cu, net GND
- removed copper zone on B.Cu, net (none)
Other:
- board text removed: "+"
- board text removed: "-"
- board text removed: "10k"
- board text removed: "24V"
- board text removed: "BME 280 BUS"
- board text removed: "NTC"
- board text removed: "SSR"
